File: Electrical/Interface-PCBA/Interface-PCBA.kicad_pcb (KiCad board)
At the start: 2 copper layers, 99.1 x 73.7 mm, 68 parts, among them J1 Conn_01x04_Male, J10 Conn_01x04_Male, J11 Conn_01x06_Male, J12 Conn_01x06_Female, J13 Conn_01x06_Female, J14 Conn_01x06_Female, J15 Conn_01x06_Female, J2 XT60-M, J3 Conn_01x02_Male, J4 Conn_01x04_Male, J5 Conn_01x04_Male, J6 Conn_01x04_Male, J7 Conn_01x06_Male, J8 Conn_01x06_Female, J9 Conn_01x06_Female, U1 LM1117-5.0

Commit message: PCB Design
Finished PCB design and sent out for fabrication
Parts:
- removed J15: Conn_01x06_Female, Connector_PinSocket_2.54mm:PinSocket_1x06_P2.54mm_Vertical
- added D1: LED, LED_SMD:LED_0603_1608Metric_Pad1.05x0.95mm_HandSolder, F.Cu at (133.4, 82.5)
- added D2: LED, LED_SMD:LED_0603_1608Metric_Pad1.05x0.95mm_HandSolder, F.Cu at (139.7, 82.5)
- added G***: LOGO, LOGO, F.Cu at (146.1, 86.4)
- added JP10: SolderJumper_2_Bridged, Jumper:SolderJumper-2_P1.3mm_Bridged_RoundedPad1.0x1.5mm, B.Cu at (122.5, 105.4)
- added JP11: SolderJumper_2_Bridged, Jumper:SolderJumper-2_P1.3mm_Bridged_RoundedPad1.0x1.5mm, B.Cu at (122.5, 102.9)
- added JP12: SolderJumper_2_Bridged, Jumper:SolderJumper-2_P1.3mm_Bridged_RoundedPad1.0x1.5mm, B.Cu at (122.5, 100.3)
- added JP13: SolderJumper_2_Bridged, Jumper:SolderJumper-2_P1.3mm_Bridged_RoundedPad1.0x1.5mm, B.Cu at (122.5, 97.8)
- added JP14: SolderJumper_2_Bridged, Jumper:SolderJumper-2_P1.3mm_Bridged_RoundedPad1.0x1.5mm, B.Cu at (108.6, 105.4)
- added JP15: SolderJumper_2_Bridged, Jumper:SolderJumper-2_P1.3mm_Bridged_RoundedPad1.0x1.5mm, B.Cu at (108.6, 108.0)
- added JP16: SolderJumper_2_Bridged, Jumper:SolderJumper-2_P1.3mm_Bridged_RoundedPad1.0x1.5mm, B.Cu at (108.6, 110.5)
- added JP17: SolderJumper_2_Bridged, Jumper:SolderJumper-2_P1.3mm_Bridged_RoundedPad1.0x1.5mm, B.Cu at (108.6, 113.0)
- added JP18: SolderJumper_2_Bridged, Jumper:SolderJumper-2_P1.3mm_Bridged_RoundedPad1.0x1.5mm, B.Cu at (108.6, 115.6)
- added JP19: SolderJumper_2_Bridged, Jumper:SolderJumper-2_P1.3mm_Bridged_RoundedPad1.0x1.5mm, B.Cu at (108.6, 90.2)
- added JP20: SolderJumper_2_Bridged, Jumper:SolderJumper-2_P1.3mm_Bridged_RoundedPad1.0x1.5mm, B.Cu at (108.6, 92.7)
- added JP21: SolderJumper_2_Bridged, Jumper:SolderJumper-2_P1.3mm_Bridged_RoundedPad1.0x1.5mm, B.Cu at (108.6, 95.2)
- added JP22: SolderJumper_2_Bridged, Jumper:SolderJumper-2_P1.3mm_Bridged_RoundedPad1.0x1.5mm, B.Cu at (108.6, 97.8)
- added JP23: SolderJumper_2_Bridged, Jumper:SolderJumper-2_P1.3mm_Bridged_RoundedPad1.0x1.5mm, B.Cu at (108.6, 100.3)
- added JP24: SolderJumper_2_Bridged, Jumper:SolderJumper-2_P1.3mm_Bridged_RoundedPad1.0x1.5mm, B.Cu at (108.6, 102.9)
- added JP7: SolderJumper_2_Bridged, Jumper:SolderJumper-2_P1.3mm_Bridged_RoundedPad1.0x1.5mm, B.Cu at (122.5, 113.0)
- added JP8: SolderJumper_2_Bridged, Jumper:SolderJumper-2_P1.3mm_Bridged_RoundedPad1.0x1.5mm, B.Cu at (122.5, 110.5)
- added JP9: SolderJumper_2_Bridged, Jumper:SolderJumper-2_P1.3mm_Bridged_RoundedPad1.0x1.5mm, B.Cu at (122.5, 108.0)
- added R14: 1k, Resistor_SMD:R_0805_2012Metric, F.Cu at (133.4, 86.4)
- added R15: 3k, Resistor_SMD:R_0805_2012Metric, F.Cu at (139.7, 86.4)
- added TP23: TestPoint, TestPoint:TestPoint_2Pads_Pitch2.54mm_Drill0.8mm, F.Cu at (76.2, 90.2)
- added TP24: TestPoint, TestPoint:TestPoint_2Pads_Pitch2.54mm_Drill0.8mm, F.Cu at (138.4, 76.2)
- added TP25: TestPoint, TestPoint:TestPoint_2Pads_Pitch2.54mm_Drill0.8mm, F.Cu at (132.1, 76.2)
- added TP26: TestPoint, TestPoint:TestPoint_2Pads_Pitch2.54mm_Drill0.8mm, F.Cu at (137.2, 125.7)
- added TP27: TestPoint, TestPoint:TestPoint_2Pads_Pitch2.54mm_Drill0.8mm, F.Cu at (142.2, 125.7)
- added TP28: TestPoint, TestPoint:TestPoint_2Pads_Pitch2.54mm_Drill0.8mm, F.Cu at (162.6, 108.0)
- added TP29: TestPoint, TestPoint:TestPoint_2Pads_Pitch2.54mm_Drill0.8mm, F.Cu at (162.6, 113.0)
- added TP30: TestPoint, TestPoint:TestPoint_2Pads_Pitch2.54mm_Drill0.8mm, F.Cu at (162.6, 118.1)
- added TP31: TestPoint, TestPoint:TestPoint_2Pads_Pitch2.54mm_Drill0.8mm, F.Cu at (162.6, 123.2)
- added TP32: TestPoint, TestPoint:TestPoint_2Pads_Pitch2.54mm_Drill0.8mm, F.Cu at (152.4, 125.7)
- added TP33: TestPoint, TestPoint:TestPoint_2Pads_Pitch2.54mm_Drill0.8mm, F.Cu at (68.6, 120.7)
- added TP34: TestPoint, TestPoint:TestPoint_2Pads_Pitch2.54mm_Drill0.8mm, F.Cu at (68.6, 115.6)
- added TP35: TestPoint, TestPoint:TestPoint_2Pads_Pitch2.54mm_Drill0.8mm, F.Cu at (68.6, 110.5)
- added TP36: TestPoint, TestPoint:TestPoint_2Pads_Pitch2.54mm_Drill0.8mm, F.Cu at (68.6, 105.4)
- J11, J2, J7: moved to B.Cu
- J14: value Conn_01x06_Female -> Conn_01x04_Male; footprint Connector_PinSocket_2.54mm:PinSocket_1x06_P2.54mm_Vertical -> Connector_JST:JST_SH_SM04B-SRSS-TB_1x04-1MP_P1.00mm_Horizontal; moved to B.Cu
- TP13, TP14, TP17, TP18, TP19, TP20, TP21, TP22: footprint TestPoint:TestPoint_Pad_D1.5mm -> TestPoint:TestPoint_2Pads_Pitch2.54mm_Drill0.8mm
- moved TP22 82.1 mm to (76.2, 86.4), turned to 180 degrees
- moved TP13 75.6 mm to (73.7, 132.1), turned to 0 degrees
- moved TP17 73.9 mm to (91.4, 120.7), turned to 0 degrees
- moved TP18 63.5 mm to (106.7, 125.7), turned to 0 degrees
- moved TP19 56.9 mm to (111.8, 125.7), turned to 0 degrees
- moved TP14 56.3 mm to (88.9, 124.5), turned to 0 degrees
- moved TP20 48.5 mm to (121.9, 125.7), turned to 0 degrees
- moved TP21 42.2 mm to (127.0, 125.7), turned to 0 degrees
- moved J14 39.2 mm to (115.6, 119.4)
- moved TP16 12.8 mm to (151.1, 76.2)
- moved TP15 12.6 mm to (144.8, 76.2)
- moved TP7 2.54 mm to (86.4, 118.1)
- moved TP9 2.54 mm to (144.8, 118.1)
- moved TP10 2.54 mm to (143.5, 120.7)
- moved TP8 2.54 mm to (86.4, 120.7)
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Connections:
- A1 pad 10: MOTOR_R_B -> Net-(A1-Pad10)
- A1 pad 11: ECHO_3 -> Net-(A1-Pad11)
- A1 pad 12: ECHO_2 -> Net-(A1-Pad12)
- A1 pad 13: ECHO_1 -> Net-(A1-Pad13)
- A1 pad 14: ENC_R_A -> Net-(A1-Pad14)
- A1 pad 15: ENC_R_B -> Net-(A1-Pad15)
- A1 pad 19: TRIG_5 -> Net-(A1-Pad19)
- A1 pad 20: TRIG_4 -> Net-(A1-Pad20)
- A1 pad 21: TRIG_3 -> Net-(A1-Pad21)
- A1 pad 22: TRIG_2 -> Net-(A1-Pad22)
- A1 pad 23: TRIG_1 -> Net-(A1-Pad23)
- A1 pad 24: ECHO_5 -> Net-(A1-Pad24)
- A1 pad 25: ECHO_4 -> Net-(A1-Pad25)
- A1 pad 5: MOTOR_L_A -> Net-(A1-Pad5)
- A1 pad 6: MOTOR_L_B -> Net-(A1-Pad6)
- A1 pad 7: ENC_L_A -> Net-(A1-Pad7)
- A1 pad 8: ENC_L_B -> Net-(A1-Pad8)
- A1 pad 9: MOTOR_R_A -> Net-(A1-Pad9)
- C1 pad 1: Net-(C1-Pad1) -> VBAT
- C3 pad 1: Net-(C1-Pad1) -> VBAT
- J3 pad 1: Net-(C1-Pad1) -> VBAT
- JP1 pad 2: Net-(C1-Pad1) -> VBAT
- R1 pad 1: Net-(C1-Pad1) -> VBAT
- TP13 pad 1: Net-(J14-Pad5) -> TRIG_1
- TP14 pad 1: Net-(J14-Pad6) -> ECHO_1
- TP17 pad 1: Net-(J15-Pad1) -> TRIG_2
- TP18 pad 1: Net-(J15-Pad2) -> ECHO_2
- TP19 pad 1: Net-(J15-Pad3) -> TRIG_3
- TP20 pad 1: Net-(J15-Pad4) -> ECHO_3
- TP21 pad 1: Net-(J15-Pad5) -> TRIG_4
- TP22 pad 1: Net-(J15-Pad6) -> VBAT
- U1 pad 3: Net-(C1-Pad1) -> VBAT
- VR1 pad 1: Net-(C1-Pad1) -> VBAT
- VR1 pad 12: Net-(C1-Pad1) -> VBAT
- VR1 pad 15: Net-(C1-Pad1) -> VBAT
- VR1 pad 16: Net-(C1-Pad1) -> VBAT
- VR1 pad 2: Net-(C1-Pad1) -> VBAT
- VR1 pad 21: Net-(C1-Pad1) -> VBAT
- VR1 pad 22: Net-(C1-Pad1) -> VBAT
Routing:
- net +3V3: track 0.00 -> 219.9 mm, vias 0 -> 11
- net +5V: track 0.00 -> 194.9 mm, vias 0 -> 8
- net +7.5V: track 0.00 -> 158.3 mm, vias 0 -> 9
- net TRIG_1: track 0.00 -> 80.4 mm, vias 0 -> 1
- net SCL: track 0.00 -> 75.5 mm, vias 0 -> 3
- net TRIG_2: track 0.00 -> 75.1 mm, vias 0 -> 1
- net ENC_L_B: track 0.00 -> 75.0 mm, vias 0 -> 3
- net ENC_L_A: track 0.00 -> 73.5 mm, vias 0 -> 3
- net SDA: track 0.00 -> 69.0 mm, vias 0 -> 3
- net ECHO_5: track 0.00 -> 67.5 mm, vias 0 -> 5
- net VBAT: track 0.00 -> 64.4 mm, vias 0 -> 2
- net MOTOR_L_B: track 0.00 -> 61.1 mm, vias 0 -> 2
- net MOTOR_L_A: track 0.00 -> 60.0 mm, vias 0 -> 2
- net TRIG_5: track 0.00 -> 58.3 mm, vias 0 -> 1
- net ECHO_4: track 0.00 -> 54.9 mm, vias 0 -> 3
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- added copper zone on B.Cu, net GND
- added copper zone on F.Cu, net GND
Other:
- board text added: "3V3"
- board text added: "5V"
- board text added: "7V"
- board text added: "BAT"
- board text added: "ESP32 Feather"
- board text added: "Mobile Robot Team: - Ellie Ko - Sofia Lopez - Liam Parrish - Austin Portinause - William Xu"
- board text added: "ON/OFF"
- board text added: "SCL"
- board text added: "SDA"
