File: Electrical/Interface-PCBA/Interface-PCBA.kicad_sch (KiCad schematic)
At the start: 68 parts, among them J1 Conn_01x04_Male, J10 Conn_01x04_Male, J11 Conn_01x06_Male, J12 Conn_01x06_Female, J13 Conn_01x06_Female, J14 Conn_01x06_Female, J15 Conn_01x06_Female, J2 XT60-M, J3 Conn_01x02_Male, J4 Conn_01x04_Male, J5 Conn_01x04_Male, J6 Conn_01x04_Male, J7 Conn_01x06_Male, J8 Conn_01x06_Female, J9 Conn_01x06_Female, U1 LM1117-5.0

Commit message: PCB Design
Finished PCB design and sent out for fabrication
Parts:
- removed J15: Conn_01x06_Female, Connector_PinSocket_2.54mm:PinSocket_1x06_P2.54mm_Vertical, symbol Connector:Conn_01x06_Female
- added D1, D2: LED, LED_SMD:LED_0603_1608Metric_Pad1.05x0.95mm_HandSolder, symbol Device:LED
- added JP10, JP11, JP12, JP13, JP14, JP15, JP16, JP17, JP18, JP19, JP20, JP21, JP22, JP23, JP24, JP7, JP8, JP9: SolderJumper_2_Bridged, Jumper:SolderJumper-2_P1.3mm_Bridged_RoundedPad1.0x1.5mm, symbol Jumper:SolderJumper_2_Bridged
- added R14: 1k, Resistor_SMD:R_0805_2012Metric, symbol Device:R
- added R15: 3k, Resistor_SMD:R_0805_2012Metric, symbol Device:R
- added TP23, TP24, TP25, TP26, TP27, TP28, TP29, TP30, TP31, TP32, TP33, TP34, TP35, TP36: TestPoint, TestPoint:TestPoint_2Pads_Pitch2.54mm_Drill0.8mm, symbol Connector:TestPoint
- J14: value Conn_01x06_Female -> Conn_01x04_Male; footprint Connector_PinSocket_2.54mm:PinSocket_1x06_P2.54mm_Vertical -> Connector_JST:JST_SH_SM04B-SRSS-TB_1x04-1MP_P1.00mm_Horizontal; symbol Connector:Conn_01x06_Female -> Connector:Conn_01x04_Male
- TP13, TP14, TP17, TP18, TP19, TP20, TP21, TP22: footprint TestPoint:TestPoint_Pad_D1.5mm -> TestPoint:TestPoint_2Pads_Pitch2.54mm_Drill0.8mm
Connections:
- net +3V3: now also D1.2 (A), TP25.1
- net +5V: now also D2.2 (A), TP24.1
- net +7.5V: now also TP23.1
- net ECHO_1: now also TP14.1, JP16.1 (A); no longer A1.13 (MISO/GPIO37)
- net ECHO_2: now also TP18.1, JP15.1 (A); no longer A1.12 (MOSI/GPIO35)
- net ECHO_3: now also TP20.1, JP14.1 (A); no longer A1.11 (SCK/GPIO36)
- net ECHO_4: now also JP13.1 (A), TP26.1; no longer A1.25 (D13/GPIO13)
- net ECHO_5: now also JP12.1 (A), TP32.1; no longer A1.24 (D12/GPIO12)
- net ENC_L_A: now also JP21.2 (B), TP29.1; no longer A1.7 (A2/GPIO16)
- net ENC_L_B: now also JP22.2 (B), TP31.1; no longer A1.8 (A3/GPIO15)
- net ENC_R_A: now also JP17.1 (A), TP34.1; no longer A1.14 (RX/GPIO38)
- net ENC_R_B: now also JP18.1 (A), TP36.1; no longer A1.15 (TX/GPIO39)
- net GND: now also R14.2, R15.2
- net MOTOR_L_A: now also JP19.2 (B); no longer A1.5 (A0/GPIO18)
- net MOTOR_L_B: now also JP20.2 (B); no longer A1.6 (A1/GPIO17)
- net MOTOR_L_NEG: now also TP30.1
- net MOTOR_L_POS: now also TP28.1
- net MOTOR_R_A: now also JP23.2 (B); no longer A1.9 (A4/GPIO14)
- net MOTOR_R_B: now also JP24.2 (B); no longer A1.10 (A5/GPIO8)
- net MOTOR_R_NEG: now also TP35.1
- net MOTOR_R_POS: now also TP33.1
- net TRIG_1: now also TP13.1, JP11.1 (A); no longer A1.23 (D11/GPIO11)
- net TRIG_2: now also TP17.1, JP10.1 (A); no longer A1.22 (D10/GPIO10)
- net TRIG_3: now also TP19.1, JP9.1 (A); no longer A1.21 (D9/GPIO9)
- net TRIG_4: now also TP21.1, JP8.1 (A); no longer A1.20 (D6/GPIO6)
- net TRIG_5: now also JP7.1 (A), TP27.1; no longer A1.19 (D5/GPIO5)
- net VBAT: now reaches TP22.1
- net VBAT: now also C1.1, C3.1, J3.1 (Pin_1), JP1.2 (B), R1.1, U1.3 (VI), VR1.1 (IN), VR1.12 (~{SHDN}), VR1.15 (IN__2), VR1.16 (IN__3), VR1.2 (IN__1), VR1.21 (IN__4), VR1.22 (IN__5)
- new net: A1.8 (A3/GPIO15), JP22.1 (A)
- new net: A1.13 (MISO/GPIO37), JP16.2 (B)
- new net: A1.10 (A5/GPIO8), JP24.1 (A)
- new net: A1.11 (SCK/GPIO36), JP14.2 (B)
- new net: A1.23 (D11/GPIO11), JP11.2 (B)
- new net: A1.12 (MOSI/GPIO35), JP15.2 (B)
- new net: A1.24 (D12/GPIO12), JP12.2 (B)
- new net: A1.21 (D9/GPIO9), JP9.2 (B)
- new net: A1.25 (D13/GPIO13), JP13.2 (B)
- new net: A1.20 (D6/GPIO6), JP8.2 (B)
- new net: D1.1 (K), R14.1
- new net: A1.9 (A4/GPIO14), JP23.1 (A)
- new net: A1.22 (D10/GPIO10), JP10.2 (B)
- new net: D2.1 (K), R15.1
- new net: A1.7 (A2/GPIO16), JP21.1 (A)
- new net: A1.14 (RX/GPIO38), JP17.2 (B)
- new net: A1.15 (TX/GPIO39), JP18.2 (B)
- new net: A1.19 (D5/GPIO5), JP7.2 (B)
- new net: A1.5 (A0/GPIO18), JP19.1 (A)
- new net: A1.6 (A1/GPIO17), JP20.1 (A)
Other:
- note added: "I^{2}C QWIIC Connect Header"
- note added: "Status LEDs"
- note removed: "IMU Socket"
- company: (none) -> W.A.L.E.S Engineering
- title: (none) -> Mobile Robot - Main PCB
- moved on the sheet: A1, H1, H2, H3, H4, J11, J12, J13, J7, J8, J9, TP1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
